File: pcb/eWeatherStation.kicad_pcb (KiCad board)
At the start: 2 copper layers, 78.3 x 48 mm, 32 parts, among them J1 SERIAL, J2 USB_B_Micro, J3 CASTELLATION, J4 1S_BATTERY, J5 RECEIVER, Q1 ZXMN3A01Z, Q2 DMC2053UVT, SW1 ENABLE, SW2 FLASH, U1 TLV75533PDBV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

Commit message: updates
Parts:
- removed R10: 100k, Resistor_SMD:R_1206_3216Metric
- R1, R14, R6: value 100k -> 150k
Connections:
- U3 pad 24: Net-(R10-Pad1) -> (no net)
- U3 pad 39: (no net) -> GND
Routing:
- net Net-(R10-Pad1): track 6.81 -> 0.00 mm

Commit message: newdesign
Parts:
- removed J1: SERIAL, !Custom:SAMTEC-TSM-103-01-X-SH
- removed Q1: ZXMN3A01Z, Package_TO_SOT_SMD:SOT-89-3_Handsoldering
- removed R1: 150k, Resistor_SMD:R_1206_3216Metric
- removed R11, R15: 10k, Resistor_SMD:R_1206_3216Metric
- removed R9: 100k, Resistor_SMD:R_1206_3216Metric
- removed SW1: ENABLE, Button_Switch_SMD:SW_SPST_PTS810
- removed SW2: FLASH, Button_Switch_SMD:SW_SPST_PTS810
- removed U3: ESP32-WROOM-32D, RF_Module:ESP32-WROOM-32
- removed U5: Si7021-A20, Package_DFN_QFN:DFN-6-1EP_3x3mm_P1mm_EP1.5x2.4mm
- added REF**: TinkerTown_Silkscreen, !Greg:TinkerTown_Silkscreen, F.Cu at (143.8, 93.2)
- added U2: ESP32-S2-WROVER, RF_Module:ESP32-S2-WROVER, F.Cu at (161.1, 72.2)
- J2: footprint Connector_USB:USB_Micro-B_Amphenol_10103594-0001LF_Horizontal -> Connector_USB:USB_Micro-B_Molex-105133-0001
- J5: value RECEIVER -> eflashy32; footprint Connector_PinSocket_2.54mm:PinSocket_1x04_P2.54mm_Vertical -> Connector_PinHeader_2.54mm:PinHeader_1x06_P2.54mm_Vertical
- moved J2 27.6 mm to (173.5, 103.8), turned to 180 degrees
- moved J5 26.8 mm to (144.7, 86.1), turned to 180 degrees
- moved C1 20.5 mm to (181.8, 88.5)
- moved U1 14.7 mm to (176.8, 88.5)
- moved R_CHG1 13.1 mm to (178.2, 97.0), turned to 270 degrees
- moved R3 11.3 mm to (160.8, 99.8)
- moved R4 10.3 mm to (160.8, 102.8), turned to 180 degrees
- moved C3 9.33 mm to (172.0, 88.5), turned to 270 degrees
- moved R2 9.28 mm to (160.8, 93.8), turned to 0 degrees
- moved C4 7.29 mm to (181.0, 104.0)
- moved U4 5.76 mm to (173.5, 97.0), turned to 270 degrees
- moved C10 3.04 mm to (169.0, 97.0), turned to 90 degrees
- moved C2 0.79 mm to (160.8, 96.8)
Connections:
- J5 pad 1: +3V3 -> GND
- J5 pad 2: /RADIO -> /TXD
- J5 pad 3: /RADIO -> /RXD
- J5 pad 4: Net-(J5-Pad4) -> +3V3
- R8 pad 1: Net-(R8-Pad1) -> /EN
Routing:
- net /SCL: track 74.1 -> 0.00 mm, vias 2 -> 0
- net /SDA: track 71.2 -> 0.00 mm, vias 2 -> 0
- net +3V3: track 133.4 -> 71.8 mm, vias 6 -> 4
- net GND: track 92.7 -> 37.1 mm, vias 15 -> 24
- net Net-(R9-Pad1): track 45.9 -> 0.00 mm, vias 2 -> 0
- net /EN: track 0.00 -> 40.8 mm, vias 0 -> 3
- net Net-(J5-Pad4): track 39.1 -> 0.00 mm
- net /RADIO: track 38.8 -> 0.00 mm, vias 1 -> 0
- net /RADIO_ENABLE: track 34.4 -> 0.00 mm
- net Net-(R8-Pad1): track 31.0 -> 0.00 mm, vias 2 -> 0
- net +BATT: track 100.7 -> 78.4 mm, vias 6 -> 4
- net /eBUSY: track 37.2 -> 58.8 mm
- net /RXD: track 55.2 -> 36.0 mm, vias 2 -> 1
- net /eDIN: track 37.7 -> 21.3 mm, vias 1 -> 3
- net Net-(J2-Pad6): track 15.0 -> 0.00 mm
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- removed copper zone on B.Cu, net GNDA
- removed copper zone on F.Cu, net GNDA
Other:
- board size 78.3 x 48 mm -> 48.8 x 48 mm
- net class Power: trace_width 0.4 -> 0.35
- board text added: "JLCJLCJLCJLCJLC"
- board text added: "eWeatherStation v2"
- board text added: "eflashy32"
